Commit message: Increase gripper and book friction, reduce book width from 3cm to 2cm

File: src/erc_description/urdf/tiago_pro.urdf (robot description, URDF)
Before this commit: robot tiago_pro, 84 links, 83 joints
Links:
- link base_antenna_left_link: geometry collision mesh filename=package://omni_base_description/meshes/base/base_antenna_li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 scale=1 1 1; visual mesh filename=package://omni_base_description/meshes/base/base_antenna_li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 scale=1 1 1
- link base_antenna_right_link: geometry collision mesh filename=package://omni_base_description/meshes/base/base_antenna_li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 scale=1 1 1; visual mesh filename=package://omni_base_description/meshes/base/base_antenna_li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 scale=1 1 1
- link suspension_front_left_link: geometry collision mesh filename=package://omni_base_description/meshes/wheels/suspension_fr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 scale=1 1 1; visual mesh filename=package://omni_base_description/meshes/wheels/suspension_fr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 scale=1 1 1
- link suspension_front_right_link: geometry collision mesh filename=package://omni_base_description/meshes/wheels/suspension_fr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 scale=1 1 1; visual mesh filename=package://omni_base_description/meshes/wheels/suspension_fr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 scale=1 1 1
- link suspension_rear_left_link: geometry collision mesh filename=package://omni_base_description/meshes/wheels/suspension_re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 scale=1 1 1; visual mesh filename=package://omni_base_description/meshes/wheels/suspension_re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 scale=1 1 1
- link suspension_rear_right_link: geometry collision mesh filename=package://omni_base_description/meshes/wheels/suspension_re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 scale=1 1 1; visual mesh filename=package://omni_base_description/meshes/wheels/suspension_re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 scale=1 1 1
- link wheel_front_left_link: geometry collision cylinder length=0.05 radius=0.0762; visual mesh filename=package://omni_base_description/meshes/wheels/wheel_link_re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 scale=1 1 1
- link wheel_front_right_link: geometry collision cylinder length=0.05 radius=0.0762; visual mesh filename=package://omni_base_description/meshes/wheels/wheel_link.stl scale=1 1 1
- link wheel_rear_left_link: geometry collision cylinder length=0.05 radius=0.0762; visual mesh filename=package://omni_base_description/meshes/wheels/wheel_link_re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 scale=1 1 1
- link wheel_rear_right_link: geometry collision cylinder length=0.05 radius=0.0762; visual mesh filename=package://omni_base_description/meshes/wheels/wheel_link.stl scale=1 1 1
Joints:
- joint gripper_left_fingertip_left_joint: limit lower=-0.1396437934520663 upper=0.7476990515543709 effort=0.1 velocity=2 -> lower=-0.1396437934520663 upper=0.7476990515543709 effort=40.0 velocity=2
- joint gripper_left_fingertip_right_joint: limit lower=-0.1396437934520663 upper=0.7476990515543709 effort=0.1 velocity=2 -> lower=-0.1396437934520663 upper=0.7476990515543709 effort=40.0 velocity=2
- joint gripper_left_inner_finger_left_joint: limit lower=-0.7476990515543709 upper=0.1396437934520663 effort=0.1 velocity=2 -> lower=-0.7476990515543709 upper=0.1396437934520663 effort=40.0 velocity=2
- joint gripper_left_inner_finger_right_joint: limit lower=-0.7476990515543709 upper=0.1396437934520663 effort=0.1 velocity=2 -> lower=-0.7476990515543709 upper=0.1396437934520663 effort=40.0 velocity=2
- joint gripper_left_outer_finger_left_joint: limit lower=-0.7476990515543709 upper=0.1396437934520663 effort=0.1 velocity=2 -> lower=-0.7476990515543709 upper=0.1396437934520663 effort=40.0 velocity=2
- joint gripper_left_outer_finger_right_joint: limit lower=-0.7476990515543709 upper=0.1396437934520663 effort=0.1 velocity=2 -> lower=-0.7476990515543709 upper=0.1396437934520663 effort=40.0 velocity=2
- joint gripper_right_fingertip_left_joint: limit lower=-0.1396437934520663 upper=0.7476990515543709 effort=0.1 velocity=2 -> lower=-0.1396437934520663 upper=0.7476990515543709 effort=40.0 velocity=2
- joint gripper_right_fingertip_right_joint: limit lower=-0.1396437934520663 upper=0.7476990515543709 effort=0.1 velocity=2 -> lower=-0.1396437934520663 upper=0.7476990515543709 effort=40.0 velocity=2
- joint gripper_right_inner_finger_left_joint: limit lower=-0.7476990515543709 upper=0.1396437934520663 effort=0.1 velocity=2 -> lower=-0.7476990515543709 upper=0.1396437934520663 effort=40.0 velocity=2
- joint gripper_right_inner_finger_right_joint: limit lower=-0.7476990515543709 upper=0.1396437934520663 effort=0.1 velocity=2 -> lower=-0.7476990515543709 upper=0.1396437934520663 effort=40.0 velocity=2
- joint gripper_right_outer_finger_left_joint: limit lower=-0.7476990515543709 upper=0.1396437934520663 effort=0.1 velocity=2 -> lower=-0.7476990515543709 upper=0.1396437934520663 effort=40.0 velocity=2
- joint gripper_right_outer_finger_right_joint: limit lower=-0.7476990515543709 upper=0.1396437934520663 effort=0.1 velocity=2 -> lower=-0.7476990515543709 upper=0.1396437934520663 effort=40.0 velocity=2

Commit message: Revert "Increase gripper and book friction, reduce book width from 3cm to 2cm"
This reverts commit 8b5f26187d17172aed8877ec4b21d8ecd239a848.

File: src/erc_description/urdf/tiago_pro.urdf (robot description, URDF)
Before this commit: robot tiago_pro, 84 links, 83 joints
Links:
- link base_antenna_left_link: geometry collision mesh filename=package://omni_base_description/meshes/base/base_antenna_li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; visual mesh filename=package://omni_base_description/meshes/base/base_antenna_li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
- link base_antenna_right_link: geometry collision mesh filename=package://omni_base_description/meshes/base/base_antenna_li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; visual mesh filename=package://omni_base_description/meshes/base/base_antenna_li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
- link suspension_front_left_link: geometry collision mesh filename=package://omni_base_description/meshes/wheels/suspension_fr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; visual mesh filename=package://omni_base_description/meshes/wheels/suspension_fr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
- link suspension_front_right_link: geometry collision mesh filename=package://omni_base_description/meshes/wheels/suspension_fr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; visual mesh filename=package://omni_base_description/meshes/wheels/suspension_fr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
- link suspension_rear_left_link: geometry collision mesh filename=package://omni_base_description/meshes/wheels/suspension_re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; visual mesh filename=package://omni_base_description/meshes/wheels/suspension_re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
- link suspension_rear_right_link: geometry collision mesh filename=package://omni_base_description/meshes/wheels/suspension_re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; visual mesh filename=package://omni_base_description/meshes/wheels/suspension_re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
- link wheel_front_left_link: geometry collision cylinder length=0.05 radius=0.0762; visual mesh filename=package://omni_base_description/meshes/wheels/wheel_link_re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
- link wheel_front_right_link: geometry collision cylinder length=0.05 radius=0.0762; visual mesh filename=package://omni_base_description/meshes/wheels/wheel_link.stl
- link wheel_rear_left_link: geometry collision cylinder length=0.05 radius=0.0762; visual mesh filename=package://omni_base_description/meshes/wheels/wheel_link_re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
- link wheel_rear_right_link: geometry collision cylinder length=0.05 radius=0.0762; visual mesh filename=package://omni_base_description/meshes/wheels/wheel_link.stl
Joints:
- joint gripper_left_fingertip_left_joint: limit lower=-0.1396437934520663 upper=0.7476990515543709 effort=40.0 velocity=2 -> lower=-0.1396437934520663 upper=0.7476990515543709 effort=0.1 velocity=2
- joint gripper_left_fingertip_right_joint: limit lower=-0.1396437934520663 upper=0.7476990515543709 effort=40.0 velocity=2 -> lower=-0.1396437934520663 upper=0.7476990515543709 effort=0.1 velocity=2
- joint gripper_left_inner_finger_left_joint: limit lower=-0.7476990515543709 upper=0.1396437934520663 effort=40.0 velocity=2 -> lower=-0.7476990515543709 upper=0.1396437934520663 effort=0.1 velocity=2
- joint gripper_left_inner_finger_right_joint: limit lower=-0.7476990515543709 upper=0.1396437934520663 effort=40.0 velocity=2 -> lower=-0.7476990515543709 upper=0.1396437934520663 effort=0.1 velocity=2
- joint gripper_left_outer_finger_left_joint: limit lower=-0.7476990515543709 upper=0.1396437934520663 effort=40.0 velocity=2 -> lower=-0.7476990515543709 upper=0.1396437934520663 effort=0.1 velocity=2
- joint gripper_left_outer_finger_right_joint: limit lower=-0.7476990515543709 upper=0.1396437934520663 effort=40.0 velocity=2 -> lower=-0.7476990515543709 upper=0.1396437934520663 effort=0.1 velocity=2
- joint gripper_right_fingertip_left_joint: limit lower=-0.1396437934520663 upper=0.7476990515543709 effort=40.0 velocity=2 -> lower=-0.1396437934520663 upper=0.7476990515543709 effort=0.1 velocity=2
- joint gripper_right_fingertip_right_joint: limit lower=-0.1396437934520663 upper=0.7476990515543709 effort=40.0 velocity=2 -> lower=-0.1396437934520663 upper=0.7476990515543709 effort=0.1 velocity=2
- joint gripper_right_inner_finger_left_joint: limit lower=-0.7476990515543709 upper=0.1396437934520663 effort=40.0 velocity=2 -> lower=-0.7476990515543709 upper=0.1396437934520663 effort=0.1 velocity=2
- joint gripper_right_inner_finger_right_joint: limit lower=-0.7476990515543709 upper=0.1396437934520663 effort=40.0 velocity=2 -> lower=-0.7476990515543709 upper=0.1396437934520663 effort=0.1 velocity=2
- joint gripper_right_outer_finger_left_joint: limit lower=-0.7476990515543709 upper=0.1396437934520663 effort=40.0 velocity=2 -> lower=-0.7476990515543709 upper=0.1396437934520663 effort=0.1 velocity=2
- joint gripper_right_outer_finger_right_joint: limit lower=-0.7476990515543709 upper=0.1396437934520663 effort=40.0 velocity=2 -> lower=-0.7476990515543709 upper=0.1396437934520663 effort=0.1 velocity=2
